File: st-nucleo-144-midi.kicad_pcb (KiCad board)
At the start: 2 copper layers, 53.3 x 77.7 mm, 4 parts, among them J1 Conn_02x08_Odd_Even, J2 Conn_02x15_Odd_Even, J3 Conn_02x10_Odd_Even, J4 Conn_02x17_Odd_Even

Commit message: Add labels to J1, J2. Update Gerber plot parameters.
Connections:
- net Net-(J1-Pad10) renamed /PC12
- net Net-(J1-Pad12) renamed /PD2
- net Net-(J1-Pad14) renamed /PG2
- net Net-(J1-Pad15) renamed /VIN
- net Net-(J1-Pad16) renamed /PG3
- net Net-(J1-Pad2) renamed /PC8
- net Net-(J1-Pad3) renamed /IOREF
- net Net-(J1-Pad4) renamed /PC9
- net Net-(J1-Pad5) renamed /NRST
- net Net-(J1-Pad6) renamed /PC10
- net Net-(J1-Pad7) renamed +3V3
- net Net-(J1-Pad8) renamed /PC11
- net Net-(J1-Pad9) renamed +5V
- net Net-(J2-Pad1) renamed /PA3
- net Net-(J2-Pad10) renamed /PD3
- net Net-(J2-Pad11) renamed /PF10
- net Net-(J2-Pad14) renamed /PE2
- net Net-(J2-Pad16) renamed /PE4
- net Net-(J2-Pad17) renamed /PF2
- net Net-(J2-Pad18) renamed /PE5
- net Net-(J2-Pad19) renamed /PF1
- net Net-(J2-Pad2) renamed /PD7
- net Net-(J2-Pad20) renamed /PE6
- net Net-(J2-Pad21) renamed /PF0
- net Net-(J2-Pad22) renamed /PE3
- net Net-(J2-Pad24) renamed /PF8
- net Net-(J2-Pad25) renamed /PD0
- net Net-(J2-Pad26) renamed /PF7
- net Net-(J2-Pad27) renamed /PD1
- net Net-(J2-Pad28) renamed /PF9
- net Net-(J2-Pad29) renamed /PG0
- net Net-(J2-Pad3) renamed /PC0
- net Net-(J2-Pad30) renamed /PG1
- net Net-(J2-Pad4) renamed /PD6
- net Net-(J2-Pad5) renamed /PC3
- net Net-(J2-Pad6) renamed /PD5
- net Net-(J2-Pad7) renamed /PF3
- net Net-(J2-Pad8) renamed /PD4
- net Net-(J2-Pad9) renamed /PF5
- J1 pad 11: Net-(J1-Pad11) -> GND
- J1 pad 13: Net-(J1-Pad13) -> GND
- J2 pad 12: Net-(J2-Pad12) -> GND
- J2 pad 23: Net-(J2-Pad23) -> GND

Commit message: Update PCB from labels, update project file to KiCad 5.0.1
Connections:
- net Net-(J3-Pad1) renamed /PC6
- net Net-(J3-Pad10) renamed /PA5
- net Net-(J3-Pad11) renamed /PC7
- net Net-(J3-Pad12) renamed /PA6
- net Net-(J3-Pad13) renamed /PB5
- net Net-(J3-Pad14) renamed /PA7
- net Net-(J3-Pad15) renamed /PB3
- net Net-(J3-Pad16) renamed /PD14
- net Net-(J3-Pad17) renamed /PA4
- net Net-(J3-Pad18) renamed /PD15
- net Net-(J3-Pad19) renamed /PB4
- net Net-(J3-Pad2) renamed /PB8
- net Net-(J3-Pad20) renamed /PF12
- net Net-(J3-Pad3) renamed /PB15
- net Net-(J3-Pad4) renamed /PB9
- net Net-(J3-Pad5) renamed /PB13
- net Net-(J3-Pad6) renamed /AREF
- net Net-(J3-Pad7) renamed /PB12
- net Net-(J3-Pad9) renamed /PA15
- net Net-(J4-Pad1) renamed VDDA
- net Net-(J4-Pad10) renamed /PE13
- net Net-(J4-Pad11) renamed /PF4
- net Net-(J4-Pad12) renamed /PF15
- net Net-(J4-Pad13) renamed /PB6
- net Net-(J4-Pad14) renamed /PG14
- net Net-(J4-Pad15) renamed /PB2
- net Net-(J4-Pad16) renamed /PG9
- net Net-(J4-Pad18) renamed /PE8
- net Net-(J4-Pad19) renamed /PD13
- net Net-(J4-Pad2) renamed /PF13
- net Net-(J4-Pad20) renamed /PE7
- net Net-(J4-Pad21) renamed /PD12
- net Net-(J4-Pad23) renamed /PD11
- net Net-(J4-Pad24) renamed /PE10
- net Net-(J4-Pad25) renamed /PE2_NC
- net Net-(J4-Pad26) renamed /PE12
- net Net-(J4-Pad29) renamed /PA0
- net Net-(J4-Pad3) renamed GNDA
- net Net-(J4-Pad30) renamed /PE15
- net Net-(J4-Pad31) renamed /PB0
- net Net-(J4-Pad32) renamed /PB10
- net Net-(J4-Pad33) renamed /PE0
- net Net-(J4-Pad34) renamed /PB11
- net Net-(J4-Pad4) renamed /PE9
- net Net-(J4-Pad6) renamed /PE11
- net Net-(J4-Pad7) renamed /PB1
- net Net-(J4-Pad9) renamed /PC2
- J3 pad 8: Net-(J3-Pad8) -> GND
- J4 pad 17: Net-(J4-Pad17) -> GND
- J4 pad 22: Net-(J4-Pad22) -> GND
- J4 pad 27: Net-(J4-Pad27) -> GND
- J4 pad 28: Net-(J4-Pad28) -> /PE14
- J4 pad 5: Net-(J4-Pad5) -> GND
- J4 pad 8: Net-(J4-Pad8) -> /PE14

Commit message: Fix misnamed pin
Connections:
- J4 pad 8: /PE14 -> /PF14
Changed lines of the file:
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@@
     (zones 0)
     (modules 4)
-    (nets 92)
+    (nets 93)
   )
   (page A4)
@@
   (net 90 /PB8)
   (net 91 /PC6)
+  (net 92 /PF14)
   (net_class Default "This is the default net class."
     (clearance 0.1524)
@@
     (add_net /PF12)
     (add_net /PF13)
+    (add_net /PF14)
     (add_net /PF15)
     (add_net /PF2)
@@
       (net 66 /PC2))
     (pad 8 thru_hole oval (at 2.54 7.62) (size 1.7 1.7) (drill 1) (layers *.Cu *.Mask)
-      (net 50 /PE14))
+      (net 92 /PF14))
     (pad 7 thru_hole oval (at 0 7.62) (size 1.7 1.7) (drill 1) (layers *.Cu *.Mask)
       (net 67 /PB1))
